Commit message: lida da'

File: test/yolobot_ws/src/yolobot_description/robot/yolobot.urdf (robot description, URDF)
Before this commit: robot yolobot, 9 links, 8 joints
Links:
- added link imu_link
- added link lidar_link, mass 0.1; collision box size=0.05 0.05 0.05; visual box size=0.05 0.05 0.05
Joints:
- added joint imu_joint: type fixed, parent chassis, child imu_link, origin xyz=0 0 0 rpy=0 0 0
- added joint lidar_joint: type fixed, parent chassis, child lidar_link, origin xyz=0.08 0 0.05 rpy=0 0 0
