Commit message: new fla

File: test/skyhunter_cpp_ws/src/yolobot_description/robot/test_bot.urdf (robot description, URDF)
Before this commit: robot agricultural_robot, 16 links, 15 joints
Links:
- removed link gps_link
- removed link left_camera_link
- removed link left_track_belt
- removed link left_track_front
- removed link left_track_middle
- removed link left_track_rear
- removed link right_camera_link
- removed link right_track_belt
- removed link right_track_front
- removed link right_track_middle
- removed link right_track_rear
- removed link sensor_mast
- removed link stereo_camera_mount
- added link chassis_link, mass 25.0; collision box size=0.8 0.5 0.2; visual box size=0.8 0.5 0.2
- added link left_wheel_front, mass 2; collision cylinder length=0.05 radius=0.1; visual cylinder length=0.05 radius=0.1
- added link left_wheel_rear, mass 2; collision cylinder length=0.05 radius=0.1; visual cylinder length=0.05 radius=0.1
- added link right_wheel_front, mass 2; collision cylinder length=0.05 radius=0.1; visual cylinder length=0.05 radius=0.1
- added link right_wheel_rear, mass 2; collision cylinder length=0.05 radius=0.1; visual cylinder length=0.05 radius=0.1
- added link sensor_head_link, mass 1.0; visual box size=0.15 0.3 0.15
- added link turret_base_link, mass 1.0; visual cylinder length=0.4 radius=0.08
- link base_link: mass 50 -> None; geometry 
- link imu_link: mass 0.1 -> None; geometry 
- link lidar_link: mass 0.5 -> None; geometry visual cylinder length=0.08 radius=0.05
Joints:
- removed joint gps_joint
- removed joint left_camera_joint
- removed joint left_track_belt_joint
- removed joint left_track_front_joint
- removed joint left_track_middle_joint
- removed joint left_track_rear_joint
- removed joint right_camera_joint
- removed joint right_track_belt_joint
- removed joint right_track_front_joint
- removed joint right_track_middle_joint
- removed joint right_track_rear_joint
- removed joint sensor_mast_joint
- removed joint stereo_camera_mount_joint
- added joint chassis_joint: type fixed, parent base_link, child chassis_link, origin xyz=0 0 0.15 rpy=0 0 0
- added joint left_wheel_front_joint: type continuous, parent chassis_link, child left_wheel_front, origin xyz=0.25 0.275 -0.05 rpy=0 0 0, axis 0 1 0
- added joint left_wheel_rear_joint: type continuous, parent chassis_link, child left_wheel_rear, origin xyz=-0.25 0.275 -0.05 rpy=0 0 0, axis 0 1 0
- added joint right_wheel_front_joint: type continuous, parent chassis_link, child right_wheel_front, origin xyz=0.25 -0.275 -0.05 rpy=0 0 0, axis 0 1 0
- added joint right_wheel_rear_joint: type continuous, parent chassis_link, child right_wheel_rear, origin xyz=-0.25 -0.275 -0.05 rpy=0 0 0, axis 0 1 0
- added joint turret_pan_joint: type revolute, parent chassis_link, child turret_base_link, origin xyz=0.2 0 0.1 rpy=0 0 0, axis 0 0 1, limit lower=-3.14 upper=3.14 effort=10 velocity=1.0
- added joint turret_tilt_joint: type revolute, parent turret_base_link, child sensor_head_link, origin xyz=0 0 0.4 rpy=0 0 0, axis 0 1 0, limit lower=-0.785 upper=0.785 effort=10 velocity=1.0
- joint imu_joint: origin xyz=0.06 0 0.2 rpy=0 0 0 -> xyz=0 0 0; parent sensor_mast -> sensor_head_link
- joint lidar_joint: origin xyz=0 0 0.26 rpy=0 0 0 -> xyz=0.05 0 0.1 rpy=0 0 0; parent sensor_mast -> sensor_head_link

File: test/skyhunter_cpp_ws/src/yolobot_description/robot/yolobot.urdf (robot description, URDF)
Before this commit: robot yolobot, 11 links, 10 joints
Links:
- removed link chassis
- removed link front_pitch_link
- removed link front_roll_link
- removed link front_yaw_link
- removed link left_wheel
- removed link rgb_cam_camera_link
- removed link rgb_cam_camera_link_frame
- removed link right_wheel
- added link chassis_link, mass 25.0; collision box size=0.8 0.5 0.15; visual box size=0.8 0.5 0.15
- added link left_wheel_front, mass 2; collision cylinder length=0.05 radius=0.1; visual cylinder length=0.05 radius=0.1
- added link left_wheel_rear, mass 2; collision cylinder length=0.05 radius=0.1; visual cylinder length=0.05 radius=0.1
- added link right_wheel_front, mass 2; collision cylinder length=0.05 radius=0.1; visual cylinder length=0.05 radius=0.1
- added link right_wheel_rear, mass 2; collision cylinder length=0.05 radius=0.1; visual cylinder length=0.05 radius=0.1
- added link sensor_head_link, mass 1.0; visual box size=0.1 0.3 0.1
- added link turret_base_link, mass 1.0; visual cylinder length=0.3 radius=0.1
- link lidar_link: mass 0.1 -> None; geometry 
Joints:
- removed joint base_link_joint
- removed joint front_pitch_joint
- removed joint front_roll_joint
- removed joint front_yaw_joint
- removed joint joint_left_wheel
- removed joint joint_right_wheel
- removed joint rgb_cam_camera_frame_joint
- removed joint rgb_cam_camera_link_joint
- added joint chassis_joint: type fixed, parent base_link, child chassis_link, origin xyz=0 0 0.1 rpy=0 0 0
- added joint left_wheel_front_joint: type continuous, parent chassis_link, child left_wheel_front, origin xyz=0.25 0.275 0, axis 0 1 0
- added joint left_wheel_rear_joint: type continuous, parent chassis_link, child left_wheel_rear, origin xyz=-0.25 0.275 0, axis 0 1 0
- added joint right_wheel_front_joint: type continuous, parent chassis_link, child right_wheel_front, origin xyz=0.25 -0.275 0, axis 0 1 0
- added joint right_wheel_rear_joint: type continuous, parent chassis_link, child right_wheel_rear, origin xyz=-0.25 -0.275 0, axis 0 1 0
- added joint turret_pan_joint: type revolute, parent chassis_link, child turret_base_link, origin xyz=0.15 0 0.2, axis 0 0 1, limit lower=-3.14 upper=3.14 effort=10 velocity=1.0
- added joint turret_tilt_joint: type revolute, parent turret_base_link, child sensor_head_link, origin xyz=0 0 0.3, axis 0 1 0, limit lower=-0.785 upper=0.785 effort=10 velocity=1.0
- joint imu_joint: origin xyz=0 0 0 rpy=0 0 0 -> xyz=0 0 0.05; parent chassis -> sensor_head_link
- joint lidar_joint: origin xyz=0.08 0 0.05 rpy=0 0 0 -> xyz=0 0 0.1; parent chassis -> sensor_head_link
