Commit message: felgw

File: test/skyhunter_swarm_ws/src/tin3_bot-0.5 .0/tin3_description/urdf/camera.xacro (robot description, xacro)
@@ -6,4 +6,6 @@
     <xacro:property name="camera_holder_z" value="0.130" />
     <xacro:property name="camera_holder_mass" value="0.3" />
+    <!-- Camera update rate: 30 (full fidelity) or 10 (optimized multi-robot) -->
+    <xacro:property name="camera_fps" value="10" />
     <!-- Namespace configuration for multi-robot support -->
     <xacro:arg name="robot_ns" default="" />
@@ -80,5 +82,5 @@
         <sensor name="rgb_camera" type="camera">
             <always_on>true</always_on>
-            <update_rate>30</update_rate>
+            <update_rate>${camera_fps}</update_rate>
             <topic>${topic_prefix}/rgb_camera/image_raw</topic>
             <gz_frame_id>${frame_prefix}rgb_camera_link</gz_frame_id>
@@ -106,5 +108,5 @@
         <sensor name="ir_camera" type="camera">
             <always_on>true</always_on>
-            <update_rate>30</update_rate>
+            <update_rate>${camera_fps}</update_rate>
             <topic>${topic_prefix}/ir_camera/image_raw</topic>
             <gz_frame_id>${frame_prefix}ir_camera_link</gz_frame_id>

File: test/skyhunter_swarm_ws/src/tin3_bot-0.5 .0/tin3_description/urdf/sensors.xacro (robot description, xacro)
@@ -123,38 +123,38 @@
     <xacro:if value="${lidar_mode != 'none'}">
         <gazebo reference="lidar_link">
-        <sensor name="lidar_sensor" type="gpu_lidar">
-        <always_on>true</always_on>
-        <update_rate>${lidar_update_rate}</update_rate>
-        <topic>${topic_prefix}/scan</topic>
-        <gz_frame_id>${frame_prefix}lidar_link</gz_frame_id>
-        <visualize>true</visualize>
-        <lidar>
-            <scan>
-            <horizontal>
-                <samples>${lidar_h_samples}</samples>
-                <resolution>1</resolution>
-                <min_angle>-2.0</min_angle>
-                <max_angle>2.0</max_angle>
-            </horizontal>
-            <vertical>
-                <samples>${lidar_v_samples}</samples>
-                <resolution>1</resolution>
-                <min_angle>-0.8</min_angle>
-                <max_angle>0.8</max_angle>
-            </vertical>
-            </scan>
-            <range>
-            <min>0.3</min>
-            <max>20.0</max>
-            <resolution>0.01</resolution>
-            </range>
-            <noise>
-            <type>gaussian</type>
-            <mean>0.0</mean>
-            <stddev>0.01</stddev>
-            </noise>
-        </lidar>
-        </sensor>
-    </gazebo>
+            <sensor name="lidar_sensor" type="gpu_lidar">
+                <always_on>true</always_on>
+                <update_rate>${lidar_update_rate}</update_rate>
+                <topic>${topic_prefix}/scan</topic>
+                <gz_frame_id>${frame_prefix}lidar_link</gz_frame_id>
+                <lidar>
+                    <scan>
+                        <horizontal>
+                            <samples>${lidar_h_samples}</samples>
+                            <resolution>1</resolution>
+                            <min_angle>-1.0472</min_angle>  <!-- -60° -->
+                            <max_angle>1.0472</max_angle>   <!-- +60° -->
+                        </horizontal>
+                        <vertical>
+                            <samples>${lidar_v_samples}</samples>
+                            <resolution>1</resolution>
+                            <min_angle>-0.7854</min_angle>  <!-- -45° -->
+                            <max_angle>0.7854</max_angle>   <!-- +45° -->
+                        </vertical>
+                    </scan>
+                    <range>
+                        <min>0.1</min>
+                        <max>30.0</max>
+                        <resolution>0.01</resolution>
+                    </range>
+                    <noise>
+                        <type>gaussian</type>
+                        <mean>0.0</mean>
+                        <stddev>0.05</stddev>  <!-- ±5cm accuracy -->
+                    </noise>
+                </lidar>
+                <visualize>true</visualize>
+            </sensor>
+        </gazebo>
     </xacro:if>
     <!-- IMU SENSOR -->
